Commit message: add sensors, add obstacles world, add initail pose to ur10

File: ur_description/urdf/ur10.urdf.xacro (robot description, xacro)
@@ -7,4 +7,6 @@
   <xacro:include filename="$(find ur_description)/urdf/ur.transmission.xacro" />
   <xacro:include filename="$(find ur_description)/urdf/ur.gazebo.xacro" />
+  <xacro:include filename="$(find ur_description)/urdf/sensors/hokuyo_utm30lx.urdf.xacro" />
+  <xacro:include filename="$(find ur_description)/urdf/sensors/_d435.urdf.xacro" />
   <xacro:macro name="cylinder_inertial" params="radius length mass *origin">
     <inertial>
@@ -277,4 +279,12 @@
       </collision>
     </link>
+    <!-- Hokuyo utm30lx-->
+    <xacro:hokuyo_utm30lx name="hokuyo" parent="${prefix}ee_link">
+      <origin xyz="0 0 0.07" rpy="0 0 0"/> <!--real measure from blue extend version-->
+    </xacro:hokuyo_utm30lx>
+    <!-- Intel realsense-->
+    <xacro:sensor_d435 parent="${prefix}ee_link">
+      <origin xyz="0.015 0 0" rpy="0 0 0"/> <!--real measure from blue extend version-->
+    </xacro:sensor_d435>
     <xacro:ur_arm_transmission prefix="${prefix}" hw_interface="${transmission_hw_interface}" />
     <xacro:ur_arm_gazebo prefix="${prefix}" />

File: ur_description/urdf/ur10_robot.urdf.xacro (robot description, xacro)
@@ -9,6 +9,5 @@
   <!-- arm -->
   <xacro:ur10_robot prefix="" joint_limited="false"
-    transmission_hw_interface="$(arg transmission_hw_interface)"
-  />
+    transmission_hw_interface="$(arg transmission_hw_interface)"/>
   <link name="world" />
   <joint name="world_joint" type="fixed">
